Commit message: Add files via upload

File: hexbot/urdf/bot_urdf.xacro (robot description, xacro)
@@ -60,5 +60,5 @@
       <origin rpy="0 0 0" xyz="0 0 0"/>
       <geometry>
-        <box size="0.01 0.06 0.03"/>
+        <box size="0.03 0.06 0.03"/>
       </geometry>
       <material name="white"/>

Commit message: Add files via upload

File: hexbot/urdf/bot_urdf.xacro (robot description, xacro)
@@ -40,4 +40,30 @@
     </visual>
   </link>
+  <link name="box_shelf">
+    <pose>0 0 0 0 0 0</pose>
+    <inertial>
+      <mass value="2"/>
+      <origin rpy="0 0 0" xyz="0 0 0"/>
+      <inertia ixx="0.0395416666667" ixy="0" ixz="0" iyy="0.106208333333" iyz="0" izz="0.106208333333"/>
+    </inertial>
+    <collision name="collision_chassis">
+      <origin rpy="0 0 0" xyz="0 0 0"/>
+      <geometry>
+        <mesh filename="package://hexbot/meshes/shell.stl" scale="1 1 1"/>
+      </geometry>
+    </collision>
+    <visual>
+      <origin rpy="0 0 0" xyz="0 0 0"/>
+      <geometry>
+        <mesh filename="package://hexbot/meshes/shell.stl" scale="1 1 1"/>
+      </geometry>
+      <material name="blue"/>
+    </visual>
+  </link>
+    <joint name="box_shelf_joint" type="fixed">
+    <origin xyz="-0.06 0 0.19" rpy="0 0 0" />
+    <parent link="link_chassis"/>
+    <child link="box_shelf" />
+  </joint>
   <!-- wheels of the bot with link, joint and transmission -->
   <xacro:wheel name="fwl" xj="0.08" yj="0.15" zj="0" />
